File: _autosave-test_pcb.kicad_pcb (KiCad board)
At the start: 2 copper layers, 55 x 70 mm, 26 parts, among them J11 Conn_01x20_Female, J8 Conn_01x20_Female, SW1 on/off switch, SW2 on/off 2

Commit message: martins whatsapp messages
Parts:
- SW2: value on/off 2 -> on/off
Changed lines of the file:
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@@
     (thickness 1.6)
     (drawings 193)
-    (tracks 255)
+    (tracks 256)
     (zones 0)
     (modules 26)
@@
     (descr "JST XH series connector, B2B-XH-A (http://www.jst-mfg.com/product/pdf/eng/eXH.pdf), generated with kicad-footprint-generator")
     (tags "connector JST XH vertical")
-    (fp_text reference led1 (at 1.25 -3.55) (layer F.SilkS)
-      (effects (font (size 1 1) (thickness 0.15)))
-    )
-    (fp_text value led (at 1.25 4.6) (layer F.Fab)
+    (fp_text reference led1 (at 1.25 -3.55) (layer F.SilkS) hide
+      (effects (font (size 1 1) (thickness 0.15)))
+    )
+    (fp_text value led (at 1.25 -3.556) (layer F.SilkS)
       (effects (font (size 1 1) (thickness 0.15)))
     )
@@
       (effects (font (size 1 1) (thickness 0.15)))
     )
-    (fp_text value "on/off 2" (at 1.25 -3.556) (layer F.SilkS)
+    (fp_text value on/off (at 1.25 -3.556) (layer F.SilkS)
       (effects (font (size 1 1) (thickness 0.15)))
     )
@@
   (segment (start 92.884 48.84236) (end 83.30636 58.42) (width 0.25) (layer B.Cu) (net 36))
   (via (at 80.772 59.944) (size 0.8) (drill 0.4) (layers F.Cu B.Cu) (net 37))
-  (segment (start 82.296 61.468) (end 80.772 59.944) (width 0.25) (layer F.Cu) (net 37))
-  (segment (start 82.296 78.74) (end 82.296 61.468) (width 0.25) (layer F.Cu) (net 37))
   (segment (start 79.756 60.96) (end 76.2 60.96) (width 0.25) (layer B.Cu) (net 37))
   (segment (start 80.772 59.944) (end 79.756 60.96) (width 0.25) (layer B.Cu) (net 37))
+  (segment (start 80.264 60.452) (end 80.772 59.944) (width 0.25) (layer F.Cu) (net 37))
+  (segment (start 80.264 76.708) (end 80.264 60.452) (width 0.25) (layer F.Cu) (net 37))
+  (segment (start 82.296 78.74) (end 80.264 76.708) (width 0.25) (layer F.Cu) (net 37))
   (segment (start 100.965 33.06) (end 100.29 33.06) (width 0.25) (layer B.Cu) (net 38))
   (segment (start 98.298 35.052) (end 98.298 44.06477) (width 0.25) (layer B.Cu) (net 38))

Commit message: added header for specific motor controller
Parts:
- removed MA1: MA, Connector_JST:JST_XH_B2B-XH-A_1x02_P2.50mm_Vertical
- removed MB1: MB, Connector_JST:JST_XH_B2B-XH-A_1x02_P2.50mm_Vertical
- removed M_power1: + motor -, TerminalBlock_Phoenix:TerminalBlock_Phoenix_MKDS-3-2-5.08_1x02_P5.08mm_Horizontal
- added mc1: Motors, Connector_PinSocket_2.54mm:PinSocket_1x06_P2.54mm_Vertical, F.Cu at (102.1, 42.7)
- moved G*** 7.91 mm to (88.6, 57.4)
- moved H3 6.93 mm to (101.9, 33.3)
- moved Servo1 5.59 mm to (82.3, 42.2)
- moved H1 1.55 mm to (67.8, 96.8)
- moved H2 1.02 mm to (61.0, 33.3)
Routing:
- net /b14: track 50.9 -> 40.2 mm
- net /b15: track 49.6 -> 39.2 mm
- net /a8: track 53.6 -> 45.3 mm
- net /b5: track 27.1 -> 20.9 mm
- net /gnd: track 304.1 -> 307.5 mm
- net /b3: track 42.7 -> 39.7 mm
- net /5v: track 227.1 -> 224.4 mm
- net (no net): track 0.00 -> 0.80 mm
