File: _autosave-test_pcb.kicad_pcb (KiCad board)
At the start: 2 copper layers, 55 x 65 mm, 37 parts, among them J1 OrangePi connector, J10 Conn_01x20_Female, J11 Conn_01x20_Female, J12 Power out, J13 Power in, J14 SRF2, J15 SRF1, J16 IR1, J17 IR2, J18 I2C2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

Commit message: breakout shema
Routing:
- net a1: track 116.6 -> 105.7 mm, vias 2 -> 1
- net a15: track 58.1 -> 64.0 mm, vias 2 -> 3
- net a3: track 62.5 -> 57.3 mm
- net 3V3: track 188.7 -> 187.1 mm
- net a4: track 10.5 -> 9.06 mm
- net b11: track 97.5 -> 98.8 mm
- net b12: track 57.5 -> 56.5 mm
- net a2: track 105.9 -> 106.7 mm
- net a0: track 101.8 -> 101.1 mm
- net a12: track 31.4 -> 32.1 mm
- net b5: track 52.6 -> 52.0 mm
- net a11: track 35.1 -> 34.6 mm
- net b4: track 44.9 -> 44.6 mm, vias 4 -> 3
- net c14: track 95.9 -> 96.1 mm, vias 5 -> 4
