File: mirte_combination.kicad_pcb (KiCad board)
At the start: 2 copper layers, 55 x 81.9 mm, 48 parts, among them J1 Servo3, J10 IR1, J11 Conn_01x13_Female, J12 IR Object Detector 1, J14 IR2, J17 MC1, J18 MC2, J19 Servo1, J2 Conn_01x20_Female, J20 SRF1, J21 ENC2, J23 MC1-A, J24 MC1-B, J25 SRF2, J26 ENC1, J27 Servo2, J28 I2C2, J3 Servo4, J30 I2C1, J33 line out left, J34 Power in, J35 Power out, J37 on/off, J4 Conn_01x20_Female, J7 Keypad, J8 Conn_01x06_Female, J9 IR Object Detector 2, Q1 DMG2305UX, Q2 DMN2050L, SW1 on/off, U1 CH340C, U2 CH340E

Commit message: v0.7: swap encoder1/2<->servo1/2 for PWM fix
Connections:
- J19 pad 3: GP2 -> GP14
- J27 pad 3: GP3 -> GP15
- R10 pad 2: GP15 -> GP2
- R11 pad 2: GP15 -> GP2
- R8 pad 2: GP14 -> GP3
- R9 pad 2: GP14 -> GP3
Routing:
- net GP2: track 74.5 -> 25.5 mm
- net GP14: track 10.9 -> 58.9 mm, vias 0 -> 1
- net GP3: track 85.3 -> 40.0 mm
- net GP15: track 73.4 -> 48.2 mm, vias 1 -> 0
- net ENC2: track 27.5 -> 29.9 mm
- net D_GND: track 62.0 -> 60.3 mm
- net 5V: track 354.5 -> 352.9 mm
- net GP1: track 49.5 -> 48.0 mm
- net 3V3: track 110.9 -> 109.4 mm
- net GP28: track 27.5 -> 26.4 mm
- net GP0: track 30.5 -> 29.4 mm
- net ECHO2: track 11.0 -> 10.2 mm
- net GP10: track 52.9 -> 52.1 mm
- net GP27: track 61.1 -> 60.4 mm
- net usb-dm3: track 38.8 -> 38.3 mm
Other:
- board text added: "v0.7"
- board text removed: "v0.6"
