File: mirte_combination.kicad_pcb (KiCad board)
At the start: 2 copper layers, 55 x 81.9 mm, 48 parts, among them J1 Servo3, J10 IR1, J11 Conn_01x13_Female, J12 IR Object Detector 1, J14 IR2, J17 MC1, J18 MC2, J19 Servo1, J2 Conn_01x20_Female, J20 SRF1, J21 ENC2, J23 MC1-A, J24 MC1-B, J25 SRF2, J26 ENC1, J27 Servo2, J28 I2C2, J3 Servo4, J30 I2C1, J33 line out left, J34 Power in, J35 Power out, J37 on/off, J4 Conn_01x20_Female, J7 Keypad, J8 Conn_01x06_Female, J9 IR Object Detector 2, Q1 DMG2305UX, Q2 DMN2050L, SW1 on/off, U1 CH340C, U2 CH340E

Commit message: adapted text, v0.8
Other:
- board text added: "v0.8"
- board text removed: "v0.7"
Changed lines of the file:
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@@
     (effects (font (size 0.8 0.8) (thickness 0.15)) (justify right mirror))
   )
-  (gr_text "GND\n" (at 154.375 131.325 270) (layer "B.SilkS")
+  (gr_text "GND\n" (at 154.37 131.42 270) (layer "B.SilkS")
     (effects (font (size 0.8 0.8) (thickness 0.15)) (justify left mirror))
   )
@@
     (effects (font (size 0.8 0.8) (thickness 0.15)) (justify mirror))
   )
-  (gr_text "5V" (at 154.425 119.7 270) (layer "B.SilkS")
+  (gr_text "5V" (at 154.42 119.85 270) (layer "B.SilkS")
     (effects (font (size 0.8 0.8) (thickness 0.15)) (justify left mirror))
   )
@@
     (effects (font (size 0.8 0.8) (thickness 0.15)) (justify right mirror))
   )
-  (gr_text "GP2" (at 154.425 117.7 270) (layer "B.SilkS")
+  (gr_text "GP14" (at 154.42 118.16 270) (layer "B.SilkS")
     (effects (font (size 0.8 0.8) (thickness 0.15)) (justify left mirror))
   )
@@
     (effects (font (size 0.8 0.8) (thickness 0.15)) (justify left mirror))
   )
-  (gr_text "GP14" (at 138.325 122.75) (layer "B.SilkS")
+  (gr_text "GP3" (at 139.12 122.71) (layer "B.SilkS")
     (effects (font (size 0.8 0.8) (thickness 0.15)) (justify right mirror))
   )
@@
     (effects (font (size 0.8 0.8) (thickness 0.15)) (justify right mirror))
   )
-  (gr_text "GP27" (at 152.05 62.2) (layer "B.SilkS")
+  (gr_text "GP16" (at 152.05 62.2) (layer "B.SilkS")
     (effects (font (size 0.8 0.8) (thickness 0.15)) (justify left mirror))
   )
@@
     (effects (font (size 0.8 0.8) (thickness 0.15)) (justify right mirror))
   )
-  (gr_text "GP15" (at 138.325 86.375) (layer "B.SilkS")
+  (gr_text "GP2" (at 139.05 86.35) (layer "B.SilkS")
     (effects (font (size 0.8 0.8) (thickness 0.15)) (justify right mirror))
   )
@@
     (effects (font (size 0.8 0.8) (thickness 0.15)) (justify right mirror))
   )
-  (gr_text "GP16" (at 152.05 69.85) (layer "B.SilkS")
+  (gr_text "GP27" (at 152.05 69.85) (layer "B.SilkS")
     (effects (font (size 0.8 0.8) (thickness 0.15)) (justify left mirror))
   )
@@
     (effects (font (size 0.8 0.8) (thickness 0.15)) (justify left mirror))
   )
-  (gr_text "5V" (at 152.05 67.25) (layer "B.SilkS")
+  (gr_text "GND" (at 152.05 67.25) (layer "B.SilkS")
     (effects (font (size 0.8 0.8) (thickness 0.15)) (justify left mirror))
   )
@@
     (effects (font (size 0.8 0.8) (thickness 0.15)) (justify left mirror))
   )
-  (gr_text "GP26" (at 152.05 72.35) (layer "B.SilkS")
+  (gr_text "GP17" (at 152.05 72.35) (layer "B.SilkS")
     (effects (font (size 0.8 0.8) (thickness 0.15)) (justify left mirror))
   )
@@
     (effects (font (size 0.8 0.8) (thickness 0.15)) (justify right mirror))
   )
-  (gr_text "GP17" (at 152.05 59.7) (layer "B.SilkS")
+  (gr_text "GP26" (at 152.05 59.7) (layer "B.SilkS")
     (effects (font (size 0.8 0.8) (thickness 0.15)) (justify left mirror))
   )
@@
     (effects (font (size 0.8 0.8) (thickness 0.15)) (justify right mirror))
   )
-  (gr_text "GND" (at 149.425 64.825) (layer "B.SilkS")
+  (gr_text "5V" (at 150.36 64.82) (layer "B.SilkS")
     (effects (font (size 0.8 0.8) (thickness 0.15)) (justify right mirror))
   )
@@
     (effects (font (size 0.8 0.8) (thickness 0.15)) (justify left mirror))
   )
-  (gr_text "5V" (at 154.4 128.4 270) (layer "B.SilkS")
+  (gr_text "5V" (at 154.39 128.51 270) (layer "B.SilkS")
     (effects (font (size 0.8 0.8) (thickness 0.15)) (justify left mirror))
   )
@@
     (effects (font (size 0.8 0.8) (thickness 0.15)) (justify right mirror))
   )
-  (gr_text "GND" (at 154.425 122.65 270) (layer "B.SilkS")
+  (gr_text "GND" (at 154.42 122.72 270) (layer "B.SilkS")
     (effects (font (size 0.8 0.8) (thickness 0.15)) (justify left mirror))
   )
@@
     (effects (font (size 0.8 0.8) (thickness 0.15)) (justify left mirror))
   )
-  (gr_text "GP3" (at 154.4 126.375 270) (layer "B.SilkS")
+  (gr_text "GP15" (at 154.39 126.43 270) (layer "B.SilkS")
     (effects (font (size 0.8 0.8) (thickness 0.15)) (justify left mirror))
   )
@@
     (effects (font (size 0.8 0.8) (thickness 0.15)))
   )
-  (gr_text "v0.7" (at 110.95 64.625) (layer "F.SilkS")
+  (gr_text "v0.8" (at 110.95 64.625) (layer "F.SilkS")
     (effects (font (size 0.8 0.8) (thickness 0.15)))
   )
