File: mirte-master/ina226.kicad_sch (KiCad schematic)
At the start: 1 part, among them J7 INA226

Commit message: First pcb design mirte master
Connections:
- net +3V3 renamed +5V
Changed lines of the file:
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@@
     )
   )
-  (symbol (lib_id "power:+3V3") (at 165.1 104.14 0) (unit 1)
+  (symbol (lib_id "power:+5V") (at 165.1 104.14 0) (unit 1)
     (in_bom yes) (on_board yes) (dnp no) (fields_autoplaced)
     (property "Reference" "#PWR017" (at 165.1 107.95 0)
       (effects (font (size 1.27 1.27)) hide)
     )
-    (property "Value" "+3V3" (at 165.1 99.06 0)
+    (property "Value" "+5V" (at 165.1 99.06 0)
       (effects (font (size 1.27 1.27)))
     )
