File: mirte-master/led_strip.kicad_sch (KiCad schematic)
At the start: 2 parts, among them J24 led_strip

Commit message: mirte-master power + start connecting pico
Parts:
- JP1: footprint (none) -> Jumper:SolderJumper-3_P1.3mm_Bridged12_RoundedPad1.0x1.5mm
Changed lines of the file:
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@@
       (effects (font (size 1.27 1.27)) (justify left))
     )
-    (property "Footprint" "" (at 96.52 71.12 0)
+    (property "Footprint" "Jumper:SolderJumper-3_P1.3mm_Bridged12_RoundedPad1.0x1.5mm" (at 96.52 71.12 0)
       (effects (font (size 1.27 1.27)) hide)
     )

Commit message: First pcb design mirte master
Parts:
- removed JP1: LED_STRIP_POWER_SELECT, Jumper:SolderJumper-3_P1.3mm_Bridged12_RoundedPad1.0x1.5mm, symbol Jumper:SolderJumper_3_Bridged12
- added JP2: LED_POWER_SELECT, Jumper:SolderJumper-3_P2.0mm_Open_TrianglePad1.0x1.5mm, symbol Jumper:Jumper_3_Open
- J24: footprint (none) -> Connector_JST:JST_XH_B3B-XH-A_1x03_P2.50mm_Vertical
Connections:
- net +12V: now also JP2.1 (A)
- net +5V: now also JP2.3 (B)
- net LED_PWR: now reaches J24.2 (Pin_2)
- net LED_PWR: now also JP2.2 (C)
Changed lines of the file:
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@@
     (stroke (width 0) (type default))
   )
-  (wire (pts (xy 110.49 68.58) (xy 113.03 68.58))
+  (wire (pts (xy 110.49 67.31) (xy 111.76 67.31))
     (stroke (width 0) (type default))
   )
-  (wire (pts (xy 90.17 80.01) (xy 90.17 81.28))
+  (wire (pts (xy 111.76 68.58) (xy 113.03 68.58))
     (stroke (width 0) (type default))
   )
@@
     (stroke (width 0) (type default))
   )
-  (wire (pts (xy 96.52 81.28) (xy 96.52 76.2))
+  (wire (pts (xy 96.52 81.28) (xy 96.52 77.47))
     (stroke (width 0) (type default))
   )
-  (wire (pts (xy 96.52 62.23) (xy 96.52 66.04))
+  (wire (pts (xy 96.52 62.23) (xy 96.52 64.77))
     (stroke (width 0) (type default))
   )
-  (wire (pts (xy 90.17 81.28) (xy 96.52 81.28))
+  (wire (pts (xy 91.44 81.28) (xy 96.52 81.28))
+    (stroke (width 0) (type default))
+  )
+  (wire (pts (xy 111.76 67.31) (xy 111.76 68.58))
     (stroke (width 0) (type default))
   )
@@
     (stroke (width 0) (type default))
   )
-  (hierarchical_label "LED_STRIP" (shape input) (at 110.49 68.58 180) (fields_autoplaced)
+  (label "LED_PWR" (at 101.6 71.12 0) (fields_autoplaced)
+    (effects (font (size 1.27 1.27)) (justify left bottom))
+  )
+  (hierarchical_label "LED_STRIP" (shape input) (at 110.49 67.31 180) (fields_autoplaced)
     (effects (font (size 1.27 1.27)) (justify right))
-  )
-  (symbol (lib_id "Jumper:SolderJumper_3_Bridged12") (at 96.52 71.12 90) (unit 1)
-    (in_bom yes) (on_board yes) (dnp no) (fields_autoplaced)
-    (property "Reference" "JP1" (at 93.98 69.85 90)
-      (effects (font (size 1.27 1.27)) (justify left))
-    )
-    (property "Value" "LED_STRIP_POWER_SELECT" (at 93.98 72.39 90)
-      (effects (font (size 1.27 1.27)) (justify left))
-    )
-    (property "Footprint" "Jumper:SolderJumper-3_P1.3mm_Bridged12_RoundedPad1.0x1.5mm" (at 96.52 71.12 0)
-      (effects (font (size 1.27 1.27)) hide)
-    )
-    (property "Datasheet" "~" (at 96.52 71.12 0)
-      (effects (font (size 1.27 1.27)) hide)
-    )
-    (pin "2")
-    (pin "1")
-    (pin "3")
-    (instances
-      (project "mirte-master"
-        (path "/19794465-0368-488c-958e-83b02754ebd6/b519899b-f03f-4ac7-8598-504888127b6d"
-          (reference "JP1") (unit 1)
-        )
-      )
-    )
   )
   (symbol (lib_id "power:+5V") (at 96.52 62.23 0) (unit 1)
@@
     )
   )
-  (symbol (lib_id "power:+12V") (at 90.17 80.01 0) (unit 1)
+  (symbol (lib_id "power:+12V") (at 91.44 81.28 0) (unit 1)
     (in_bom yes) (on_board yes) (dnp no) (fields_autoplaced)
-    (property "Reference" "#PWR054" (at 90.17 83.82 0)
+    (property "Reference" "#PWR054" (at 91.44 85.09 0)
       (effects (font (size 1.27 1.27)) hide)
     )
-    (property "Value" "+12V" (at 90.17 74.93 0)
+    (property "Value" "+12V" (at 91.44 76.2 0)
       (effects (font (size 1.27 1.27)))
     )
-    (property "Footprint" "" (at 90.17 80.01 0)
+    (property "Footprint" "" (at 91.44 81.28 0)
       (effects (font (size 1.27 1.27)) hide)
     )
-    (property "Datasheet" "" (at 90.17 80.01 0)
+    (property "Datasheet" "" (at 91.44 81.28 0)
       (effects (font (size 1.27 1.27)) hide)
     )
@@
       (effects (font (size 1.27 1.27)) (justify left))
     )
-    (property "Footprint" "" (at 118.11 71.12 0)
+    (property "Footprint" "Connector_JST:JST_XH_B3B-XH-A_1x03_P2.50mm_Vertical" (at 118.11 71.12 0)
       (effects (font (size 1.27 1.27)) hide)
     )
@@
         )
       )
+    )
+  )
+  (symbol (lib_id "Jumper:Jumper_3_Open") (at 96.52 71.12 90) (unit 1)
+    (in_bom yes) (on_board yes) (dnp no) (fields_autoplaced)
+    (property "Reference" "JP2" (at 93.98 69.85 90)
+      (effects (font (size 1.27 1.27)) (justify left))
+    )
+    (property "Value" "LED_POWER_SELECT" (at 93.98 72.39 90)
+      (effects (font (size 1.27 1.27)) (justify left))
+    )
+    (property "Footprint" "Jumper:SolderJumper-3_P2.0mm_Open_TrianglePad1.0x1.5mm" (at 96.52 71.12 0)
+      (effects (font (size 1.27 1.27)) hide)
+    )
+    (property "Datasheet" "~" (at 96.52 71.12 0)
+      (effects (font (size 1.27 1.27)) hide)
+    )
+    (pin "3")
+    (pin "1")
+    (pin "2")
+    (instances
+      (project "mirte-master"
+        (path "/19794465-0368-488c-958e-83b02754ebd6/b519899b-f03f-4ac7-8598-504888127b6d"
+          (reference "JP2") (unit 1)
+        )
+      )
