File: mirte-master/motor.kicad_sch (KiCad schematic)
At the start: 1 part, among them J11 encoder_motor

Commit message: First pcb design mirte master
Connections:
- net VCC renamed +3V3
Changed lines of the file:
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@@
     (effects (font (size 1.27 1.27)) (justify right))
-  )
-  (symbol (lib_id "power:VCC") (at 109.22 97.79 0) (unit 1)
-    (in_bom yes) (on_board yes) (dnp no) (fields_autoplaced)
-    (property "Reference" "#PWR026" (at 109.22 101.6 0)
-      (effects (font (size 1.27 1.27)) hide)
-    )
-    (property "Value" "VCC" (at 109.22 92.71 0)
-      (effects (font (size 1.27 1.27)))
-    )
-    (property "Footprint" "" (at 109.22 97.79 0)
-      (effects (font (size 1.27 1.27)) hide)
-    )
-    (property "Datasheet" "" (at 109.22 97.79 0)
-      (effects (font (size 1.27 1.27)) hide)
-    )
-    (pin "1")
-    (instances
-      (project "mirte-master"
-        (path "/19794465-0368-488c-958e-83b02754ebd6/51f438bb-e502-4544-ae45-b231cb2dc289/1618e457-71da-404d-b24b-344883770d69"
-          (reference "#PWR026") (unit 1)
-        )
-        (path "/19794465-0368-488c-958e-83b02754ebd6/51f438bb-e502-4544-ae45-b231cb2dc289/172e9393-c3bf-49f7-b8ed-9f9e42b81e17"
-          (reference "#PWR028") (unit 1)
-        )
-        (path "/19794465-0368-488c-958e-83b02754ebd6/51f438bb-e502-4544-ae45-b231cb2dc289/2206942f-8827-462d-8b4e-ac2211508605"
-          (reference "#PWR030") (unit 1)
-        )
-        (path "/19794465-0368-488c-958e-83b02754ebd6/51f438bb-e502-4544-ae45-b231cb2dc289/09f04b0c-9443-45a0-adc5-c663013664a2"
-          (reference "#PWR032") (unit 1)
-        )
-      )
-    )
   )
   (symbol (lib_id "power:GND") (at 109.22 74.93 0) (unit 1)
@@
         )
       )
+    )
+  )
+  (symbol (lib_id "power:+3V3") (at 109.22 97.79 0) (unit 1)
+    (in_bom yes) (on_board yes) (dnp no) (fields_autoplaced)
+    (property "Reference" "#PWR026" (at 109.22 101.6 0)
+      (effects (font (size 1.27 1.27)) hide)
+    )
+    (property "Value" "+3V3" (at 109.22 92.71 0)
+      (effects (font (size 1.27 1.27)))
+    )
+    (property "Footprint" "" (at 109.22 97.79 0)
+      (effects (font (size 1.27 1.27)) hide)
+    )
+    (property "Datasheet" "" (at 109.22 97.79 0)
+      (effects (font (size 1.27 1.27)) hide)
+    )
+    (pin "1")
+    (instances
+      (project "mirte-master"
+        (path "/19794465-0368-488c-958e-83b02754ebd6/51f438bb-e502-4544-ae45-b231cb2dc289/1618e457-71da-404d-b24b-344883770d69"
+          (reference "#PWR026") (unit 1)
+        )
+        (path "/19794465-0368-488c-958e-83b02754ebd6/51f438bb-e502-4544-ae45-b231cb2dc289/172e9393-c3bf-49f7-b8ed-9f9e42b81e17"
+          (reference "#PWR028") (unit 1)
+        )
+        (path "/19794465-0368-488c-958e-83b02754ebd6/51f438bb-e502-4544-ae45-b231cb2dc289/2206942f-8827-462d-8b4e-ac2211508605"
+          (reference "#PWR030") (unit 1)
+        )
+        (path "/19794465-0368-488c-958e-83b02754ebd6/51f438bb-e502-4544-ae45-b231cb2dc289/09f04b0c-9443-45a0-adc5-c663013664a2"
+          (reference "#PWR032") (unit 1)
+        )
+      )
