File: mirte-master/motor.kicad_sch (KiCad schematic)
At the start: 1 part, among them J11 encoder_motor

Commit message: Add bottom pcb mirte-master
Parts:
- renumbered J11 to #J11
Changed lines of the file:
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@@
   (symbol (lib_id "Connector:Conn_01x04_Socket") (at 120.65 85.09 0) (unit 1)
     (in_bom yes) (on_board yes) (dnp no) (fields_autoplaced)
-    (property "Reference" "J11" (at 121.92 85.09 0)
+    (property "Reference" "#J11" (at 121.92 85.09 0)
       (effects (font (size 1.27 1.27)) (justify left))
     )
@@
       (project "mirte-master"
         (path "/19794465-0368-488c-958e-83b02754ebd6/51f438bb-e502-4544-ae45-b231cb2dc289/1618e457-71da-404d-b24b-344883770d69"
-          (reference "J11") (unit 1)
+          (reference "#J11") (unit 1)
         )
         (path "/19794465-0368-488c-958e-83b02754ebd6/51f438bb-e502-4544-ae45-b231cb2dc289/172e9393-c3bf-49f7-b8ed-9f9e42b81e17"
-          (reference "J12") (unit 1)
+          (reference "#J12") (unit 1)
         )
         (path "/19794465-0368-488c-958e-83b02754ebd6/51f438bb-e502-4544-ae45-b231cb2dc289/2206942f-8827-462d-8b4e-ac2211508605"
-          (reference "J13") (unit 1)
+          (reference "#J13") (unit 1)
         )
         (path "/19794465-0368-488c-958e-83b02754ebd6/51f438bb-e502-4544-ae45-b231cb2dc289/09f04b0c-9443-45a0-adc5-c663013664a2"
-          (reference "J14") (unit 1)
+          (reference "#J14") (unit 1)
         )
       )
