File: mirte-master/5vreg.kicad_sch (KiCad schematic)
At the start: 1 part, among them J21 5v_regulator

Commit message: First pcb design mirte master
Parts:
- J21: footprint (none) -> TerminalBlock_Phoenix:TerminalBlock_Phoenix_PT-1,5-4-5.0-H_1x04_P5.00mm_Horizontal
Changed lines of the file:
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@@
 (kicad_sch (version 20230121) (generator eeschema)
   (paper "A4")
+  (junction (at 105.41 87.63) (diameter 0) (color 0 0 0 0)
+  )
   (wire (pts (xy 118.11 78.74) (xy 118.11 82.55))
     (stroke (width 0) (type default))
@@
     (stroke (width 0) (type default))
   )
+  (wire (pts (xy 105.41 87.63) (xy 119.38 87.63))
+    (stroke (width 0) (type default))
+  )
   (wire (pts (xy 116.84 90.17) (xy 119.38 90.17))
     (stroke (width 0) (type default))
@@
     (stroke (width 0) (type default))
   )
-  (wire (pts (xy 105.41 87.63) (xy 119.38 87.63))
+  (wire (pts (xy 97.79 87.63) (xy 105.41 87.63))
     (stroke (width 0) (type default))
   )
@@
       (effects (font (size 1.27 1.27)) (justify left))
     )
-    (property "Footprint" "" (at 124.46 85.09 0)
+    (property "Footprint" "TerminalBlock_Phoenix:TerminalBlock_Phoenix_PT-1,5-4-5.0-H_1x04_P5.00mm_Horizontal" (at 124.46 85.09 0)
       (effects (font (size 1.27 1.27)) hide)
     )
@@
     )
   )
-  (symbol (lib_id "power:+5V") (at 105.41 87.63 0) (unit 1)
+  (symbol (lib_id "power:+5V") (at 97.79 87.63 0) (unit 1)
     (in_bom yes) (on_board yes) (dnp no) (fields_autoplaced)
-    (property "Reference" "#PWR045" (at 105.41 91.44 0)
+    (property "Reference" "#PWR045" (at 97.79 91.44 0)
       (effects (font (size 1.27 1.27)) hide)
     )
-    (property "Value" "+5V" (at 105.41 82.55 0)
+    (property "Value" "+5V" (at 97.79 82.55 0)
       (effects (font (size 1.27 1.27)))
     )
-    (property "Footprint" "" (at 105.41 87.63 0)
+    (property "Footprint" "" (at 97.79 87.63 0)
       (effects (font (size 1.27 1.27)) hide)
     )
-    (property "Datasheet" "" (at 105.41 87.63 0)
+    (property "Datasheet" "" (at 97.79 87.63 0)
       (effects (font (size 1.27 1.27)) hide)
     )
@@
         )
       )
+    )
+  )
+  (symbol (lib_id "power:PWR_FLAG") (at 105.41 87.63 0) (unit 1)
+    (in_bom yes) (on_board yes) (dnp no) (fields_autoplaced)
+    (property "Reference" "#FLG04" (at 105.41 85.725 0)
+      (effects (font (size 1.27 1.27)) hide)
+    )
+    (property "Value" "PWR_FLAG" (at 105.41 82.55 0)
+      (effects (font (size 1.27 1.27)))
+    )
+    (property "Footprint" "" (at 105.41 87.63 0)
+      (effects (font (size 1.27 1.27)) hide)
+    )
+    (property "Datasheet" "~" (at 105.41 87.63 0)
+      (effects (font (size 1.27 1.27)) hide)
+    )
+    (pin "1")
+    (instances
+      (project "mirte-master"
+        (path "/19794465-0368-488c-958e-83b02754ebd6/17ebe4c8-09bb-4699-976c-396d27e4a3f5/1f6ba3bd-b93c-4e80-aba0-1409dab869f7"
+          (reference "#FLG04") (unit 1)
+        )
+      )

Commit message: updates master, holes, components
Connections:
- net +12V: now also J21.4 (Pin_4); no longer J21.1 (Pin_1)
- net +5V: now also J21.2 (Pin_2); no longer J21.3 (Pin_3)
- net GND: now also J21.1 (Pin_1), J21.3 (Pin_3); no longer J21.2 (Pin_2), J21.4 (Pin_4)
Changed lines of the file:
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@@
     )
   )
-  (symbol (lib_id "Connector:Screw_Terminal_01x04") (at 124.46 85.09 0) (unit 1)
-    (in_bom yes) (on_board yes) (dnp no) (fields_autoplaced)
-    (property "Reference" "J21" (at 127 85.09 0)
+  (symbol (lib_id "Connector:Screw_Terminal_01x04") (at 124.46 87.63 0) (mirror x) (unit 1)
+    (in_bom yes) (on_board yes) (dnp no)
+    (property "Reference" "J21" (at 127 87.63 0)
       (effects (font (size 1.27 1.27)) (justify left))
     )
-    (property "Value" "5v_regulator" (at 127 87.63 0)
+    (property "Value" "5v_regulator" (at 127 85.09 0)
       (effects (font (size 1.27 1.27)) (justify left))
     )
-    (property "Footprint" "TerminalBlock_Phoenix:TerminalBlock_Phoenix_PT-1,5-4-5.0-H_1x04_P5.00mm_Horizontal" (at 124.46 85.09 0)
+    (property "Footprint" "TerminalBlock_Phoenix:TerminalBlock_Phoenix_PT-1,5-4-5.0-H_1x04_P5.00mm_Horizontal" (at 124.46 87.63 0)
       (effects (font (size 1.27 1.27)) hide)
     )
-    (property "Datasheet" "~" (at 124.46 85.09 0)
+    (property "Datasheet" "~" (at 124.46 87.63 0)
       (effects (font (size 1.27 1.27)) hide)
     )
