File: mirte-master/hbridge_power.kicad_sch (KiCad schematic)
At the start: 2 parts, among them J22 hbridge_1, J23 hbridge_2

Commit message: First pcb design mirte master
Parts:
- J22, J23: footprint (none) -> TerminalBlock_Phoenix:TerminalBlock_Phoenix_PT-1,5-2-5.0-H_1x02_P5.00mm_Horizontal
Changed lines of the file:
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@@
       (effects (font (size 1.27 1.27)) (justify left))
     )
-    (property "Footprint" "" (at 116.84 72.39 0)
+    (property "Footprint" "TerminalBlock_Phoenix:TerminalBlock_Phoenix_PT-1,5-2-5.0-H_1x02_P5.00mm_Horizontal" (at 116.84 72.39 0)
       (effects (font (size 1.27 1.27)) hide)
     )
@@
       (effects (font (size 1.27 1.27)) (justify left))
     )
-    (property "Footprint" "" (at 116.84 93.98 0)
+    (property "Footprint" "TerminalBlock_Phoenix:TerminalBlock_Phoenix_PT-1,5-2-5.0-H_1x02_P5.00mm_Horizontal" (at 116.84 93.98 0)
       (effects (font (size 1.27 1.27)) hide)
     )

Commit message: add lcsc libs
Parts:
- J22, J23: footprint TerminalBlock_Phoenix:TerminalBlock_Phoenix_PT-1,5-2-5.0-H_1x02_P5.00mm_Horizontal -> easyeda:CONN-TH_XY126V-5.0-2P
Changed lines of the file:
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@@
       (effects (font (size 1.27 1.27)) (justify left))
     )
-    (property "Footprint" "TerminalBlock_Phoenix:TerminalBlock_Phoenix_PT-1,5-2-5.0-H_1x02_P5.00mm_Horizontal" (at 116.84 72.39 0)
+    (property "Footprint" "easyeda:CONN-TH_XY126V-5.0-2P" (at 116.84 72.39 0)
       (effects (font (size 1.27 1.27)) hide)
     )
@@
       (effects (font (size 1.27 1.27)) (justify left))
     )
-    (property "Footprint" "TerminalBlock_Phoenix:TerminalBlock_Phoenix_PT-1,5-2-5.0-H_1x02_P5.00mm_Horizontal" (at 116.84 93.98 0)
+    (property "Footprint" "easyeda:CONN-TH_XY126V-5.0-2P" (at 116.84 93.98 0)
       (effects (font (size 1.27 1.27)) hide)
     )
